File: drone/drone.sch (KiCad schematic (older format))
At the start: 30 parts, among them IC1 AT89S4051-P, P1 CONN_2, P2 ISP, P3 CONN_2, P4 Blade1, P5 Blade2, Q1 NPN, Q2 PNP, Q3 NPN, Q4 PNP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

Commit message: Associated parts in the netlist
Parts:
- added Q9: NPN, symbol NPN
- added R9: 3K3, symbol R
- P1: value CONN_2 -> LeftM
- P3: value CONN_2 -> RightM
Connections:
- net labels added: BladeCon
- wire segments 88 -> 92
- no-connect marks 8 -> 7
Changed lines of the file:
@@
 	7200 1825 7050 1825
 Connection ~ 7050 1825
-$Comp
-L +12V #PWR09
-U 1 1 556F2BC6
-P 7125 1075
-F 0 "#PWR09" H 7125 1025 20  0001 C CNN
-F 1 "+12V" H 7125 1175 30  0000 C CNN
-F 2 "" H 7125 1075 60  0000 C CNN
-F 3 "" H 7125 1075 60  0000 C CNN
-	1    7125 1075
-	1    0    0    -1
-$EndComp
 Wire Wire Line
 	7125 1075 7125 1625
@@
 $EndComp
 $Comp
-L +12V #PWR010
+L +12V #PWR09
 U 1 1 556F3087
 P 8575 2250
-F 0 "#PWR010" H 8575 2200 20  0001 C CNN
+F 0 "#PWR09" H 8575 2200 20  0001 C CNN
 F 1 "+12V" H 8575 2350 30  0000 C CNN
 F 2 "" H 8575 2250 60  0000 C CNN
@@
 $EndComp
 $Comp
-L +5V #PWR011
+L +5V #PWR010
 U 1 1 556F309B
 P 9625 2300
-F 0 "#PWR011" H 9625 2390 20  0001 C CNN
+F 0 "#PWR010" H 9625 2390 20  0001 C CNN
 F 1 "+5V" H 9625 2390 30  0000 C CNN
 F 2 "" H 9625 2300 60  0000 C CNN
@@
 $EndComp
 $Comp
-L GND #PWR012
+L GND #PWR011
 U 1 1 556F30B9
 P 8400 2975
-F 0 "#PWR012" H 8400 2975 30  0001 C CNN
+F 0 "#PWR011" H 8400 2975 30  0001 C CNN
 F 1 "GND" H 8400 2905 30  0001 C CNN
 F 2 "" H 8400 2975 60  0000 C CNN
@@
 P 3250 4450
 F 0 "P1" V 3200 4450 40  0000 C CNN
-F 1 "CONN_2" V 3300 4450 40  0000 C CNN
+F 1 "LeftM" V 3300 4450 40  0000 C CNN
 F 2 "" H 3250 4450 60  0000 C CNN
 F 3 "" H 3250 4450 60  0000 C CNN
@@
 	2850 5275 3625 5275
 $Comp
-L GND #PWR013
+L GND #PWR012
 U 1 1 556F5C27
 P 3250 5375
-F 0 "#PWR013" H 3250 5375 30  0001 C CNN
+F 0 "#PWR012" H 3250 5375 30  0001 C CNN
 F 1 "GND" H 3250 5305 30  0001 C CNN
 F 2 "" H 3250 5375 60  0000 C CNN
@@
 $EndComp
 $Comp
-L +12V #PWR014
+L +12V #PWR013
 U 1 1 556F5C3B
 P 3250 4200
-F 0 "#PWR014" H 3250 4150 20  0001 C CNN
+F 0 "#PWR013" H 3250 4150 20  0001 C CNN
 F 1 "+12V" H 3250 4300 30  0000 C CNN
 F 2 "" H 3250 4200 60  0000 C CNN
@@
 P 7300 4450
 F 0 "P3" V 7250 4450 40  0000 C CNN
-F 1 "CONN_2" V 7350 4450 40  0000 C CNN
+F 1 "RightM" V 7350 4450 40  0000 C CNN
 F 2 "" H 7300 4450 60  0000 C CNN
 F 3 "" H 7300 4450 60  0000 C CNN
@@
 	6900 5275 7675 5275
 $Comp
-L GND #PWR015
+L GND #PWR014
 U 1 1 556F617A
 P 7300 5375
-F 0 "#PWR015" H 7300 5375 30  0001 C CNN
+F 0 "#PWR014" H 7300 5375 30  0001 C CNN
 F 1 "GND" H 7300 5305 30  0001 C CNN
 F 2 "" H 7300 5375 60  0000 C CNN
@@
 Int0
 $Comp
-L +12V #PWR016
+L +12V #PWR015
 U 1 1 556F628D
 P 7300 4200
-F 0 "#PWR016" H 7300 4150 20  0001 C CNN
+F 0 "#PWR015" H 7300 4150 20  0001 C CNN
 F 1 "+12V" H 7300 4300 30  0000 C CNN
 F 2 "" H 7300 4200 60  0000 C CNN
@@
 Wire Wire Line
 	4275 1675 4350 1675
-NoConn ~ 4275 1775
 NoConn ~ 4275 1475
 NoConn ~ 4275 1375
 NoConn ~ 4275 2375
 NoConn ~ 4275 2675
+Text GLabel 4350 1775 2    60   Input ~ 0
+BladeCon
+Wire Wire Line
+	4275 1775 4350 1775
+$Comp
+L +12V #PWR016
+U 1 1 556F6D84
+P 7125 625
+F 0 "#PWR016" H 7125 575 20  0001 C CNN
+F 1 "+12V" H 7125 725 30  0000 C CNN
+F 2 "" H 7125 625 60  0000 C CNN
+F 3 "" H 7125 625 60  0000 C CNN
+	1    7125 625
+	1    0    0    -1
+$EndComp
+$Comp
+L NPN Q9
+U 1 1 556F6D98
+P 7025 875
+F 0 "Q9" H 7025 725 50  0000 R CNN
+F 1 "NPN" H 7025 1025 50  0000 R CNN
+F 2 "" H 7025 875 60  0000 C CNN
+F 3 "" H 7025 875 60  0000 C CNN
+	1    7025 875
+	1    0    0    -1
+$EndComp
+Wire Wire Line
+	7125 675  7125 625
+Text GLabel 6250 875  0    60   Input ~ 0
+BladeCon
+Wire Wire Line
+	6775 875  6825 875
+$Comp
+L R R9
+U 1 1 556F6198
+P 6525 875
+F 0 "R9" V 6605 875 40  0000 C CNN
+F 1 "3K3" V 6532 876 40  0000 C CNN
+F 2 "" V 6455 875 30  0000 C CNN
+F 3 "" H 6525 875 30  0000 C CNN
+	1    6525 875
+	0    1    1    0
+$EndComp
+Wire Wire Line
+	6250 875  6275 875
 $EndSCHEMATC
