File: drone/drone.kicad_pcb (KiCad board)
At the start: 2 copper layers, 58.4 x 73 mm, 32 parts, among them IC1 AT89S4051-P, P1 LeftM, P2 ISP, P3 RightM, P4 Blade1, P5 Blade2, Q1 NPN, Q2 PNP, Q3 NPN, Q4 PNP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

Commit message: Revised the PCB design
* Set the board outlines
* Worked on the message text
Parts:
- moved SW2 2.50 mm to (170.2, 76.2)
Routing:
- net Net-(P1-Pad1): track 39.4 -> 97.0 mm, vias 1 -> 3
- net Reset: track 36.0 -> 46.2 mm, vias 2 -> 1
- net RMotor2: track 61.7 -> 66.6 mm, vias 3 -> 6
- net +12V: track 92.0 -> 96.3 mm
- net Int0: track 39.3 -> 36.2 mm
- net GND: track 160.0 -> 162.6 mm
- net Net-(P3-Pad1): track 36.2 -> 37.7 mm
- net RMotor1: track 55.0 -> 56.4 mm
- net BladeCon: track 28.1 -> 29.4 mm
- net LMotor1: track 51.0 -> 52.3 mm, vias 3 -> 2
- net LMotor2: track 66.7 -> 65.6 mm, vias 2 -> 0
- net Net-(P3-Pad2): track 24.1 -> 25.2 mm, vias 1 -> 0
- net Net-(IC1-Pad18): track 11.6 -> 12.2 mm
- net Net-(P4-Pad1): track 28.8 -> 28.3 mm
- net Net-(P1-Pad2): track 27.4 -> 27.6 mm, vias 1 -> 0
Other:
- board size 58.4 x 73 mm -> 62.5 x 72 mm
- board text added: "(c)2015 Henry Schmale"
- board text removed: "MowerDrone rev 0.1"
